Commit message: Initial clean ROS2 project (removed build/install/log/vscode)

File: src/ros_project/description/robot.urdf.xacro (robot description, xacro)
@@ -3,3 +3,4 @@
     <!-- Example link -->
     <xacro:include filename="$(find ros_project)/description/robot_core.xacro"/>
+    <xacro:include filename="$(find ros_project)/description/lidar.xacro"/>
 </robot>

File: src/ros_project/description/robot_core.xacro (robot description, xacro)
@@ -5,25 +5,44 @@
     filename="libgz-sim-diff-drive-system.so"
     name="gz::sim::systems::DiffDrive">
-    <!-- Wheel joints -->
-    <left_joint>left_wheel_joint</left_joint>
-    <right_joint>right_wheel_joint</right_joint>
-    <!-- Geometry -->
-    <wheel_separation>0.4</wheel_separation>
-    <wheel_radius>0.05</wheel_radius>
-    <!-- Topics -->
-    <topic>cmd_vel</topic>
-    <odometry_topic>odom</odometry_topic>
-    <odometry_frame>odom</odometry_frame>
-    <robot_base_frame>base_link</robot_base_frame>
-    <!-- Motion limits -->
-    <max_linear_velocity>1.0</max_linear_velocity>
-    <max_angular_velocity>2.0</max_angular_velocity>
-    <!-- Debug -->
-    <print_msgs>true</print_msgs>
+        <!--Wheel information -->
+        <left_joint>left_wheel_joint</left_joint>
+        <right_joint>right_wheel_joint</right_joint>
+        <wheel_separation>0.35</wheel_separation>
+        <wheel_radius>0.05</wheel_radius>
+        <!-- limits -->
+        <max_wheel_torque>200</max_wheel_torque>
+        <max_wheel_acceleration>10.0</max_wheel_acceleration>
+        <frame_id>odom</frame_id>
+        <child_frame_id>base_link</child_frame_id>
+        <tf_topic>/tf</tf_topic>
+        <odom_topic>/odom</odom_topic>
+        <!-- outputs-->
+        <robot_base_frame>base_link</robot_base_frame>
+        <!-- topics-->
+        <topic>cmd_vel</topic>
+        <publish_odom>true</publish_odom>
+        <publish_odom_tf>true</publish_odom_tf>
+        <publish_wheel_tf>true</publish_wheel_tf>
   </plugin>
+  <plugin
+    filename="libgz-sim-joint-state-publisher-system.so"
+    name="gz::sim::systems::JointStatePublisher">
+    <topic>/joint_states</topic>
+  </plugin>
+</gazebo>
+<gazebo reference="caster_wheel">
+  <mu1 value="0.1"/>
+  <mu2 value="0.1"/>
 </gazebo>
 <xacro:include filename="inertial_macros.xacro"/>
 <!-- Base link -->
 <link name = "base_link">
+</link>
+<joint name="base_footprint_joint" type="fixed">
+  <parent link="base_link"/>
+  <child link="base_footprint"/>
+  <origin xyz="0 0 0" rpy="0 0 0"/>
+</joint>
+<link name="base_footprint">
 </link>
 <!--Chassis-->
@@ -105,29 +124,4 @@
     </xacro:inertial_cylinder>
 </link>
-<joint name  = "lidar_joint" type = "fixed">
-    <parent link = "chassis"/>
-    <child link = "lidar_link"/>
-    <origin xyz = "0.1 0 0" rpy = "0 0 0"/>
-</joint>
-<link name = "lidar_link">
-    <visual>
-        <origin xyz = "0.1 0 0.1"/>
-        <geometry>
-            <sphere radius = "0.02"/>
-        </geometry>
-        <material name = "green">
-            <color rgba = "0 1 0 1"/>
-        </material>
-    </visual>
-    <collision>
-        <origin xyz = "0.1 0 0.1"/>
-        <geometry>
-            <sphere radius = "0.02"/>
-        </geometry>
-    </collision>
-    <xacro:inertial_sphere mass = "0.01" radius="0.02">
-        <origin xyz ="0.1 0 0.1"/>
-    </xacro:inertial_sphere>
-</link>
 <joint name  = "casterwheel" type = "fixed">
     <parent link = "chassis"/>
