Commit message: hi

File: src/ros_project/urdf/slam_lidar_midplate_front.xacro (robot description, xacro)
@@ -1,7 +1,7 @@
 <?xml version="1.0" ?>
-<robot name="slam" xmlns:xacro="http://www.ros.org/wiki/xacro">
+<robot name="slam_lidar_midplate_front" xmlns:xacro="http://www.ros.org/wiki/xacro">
 <xacro:include filename="$(find ros_project)/urdf/materials.xacro" />
-<xacro:include filename="$(find ros_project)/urdf/slam.ros2control" />
-<xacro:include filename="$(find ros_project)/urdf/slam.gazebo" />
+<xacro:include filename="$(find ros_project)/urdf/slam_lidar_midplate_front.ros2control" />
+<xacro:include filename="$(find ros_project)/urdf/slam_lidar_midplate_front.gazebo" />
 <gazebo>
   <plugin
@@ -15,15 +15,20 @@
     <tf_topic>/tf</tf_topic>
     <frame_id>odom</frame_id>
-    <child_frame_id>base_link</child_frame_id>
+    <child_frame_id>base_footprint</child_frame_id>
     <topic>cmd_vel</topic>
     <publish_odom>true</publish_odom>
     <publish_odom_tf>true</publish_odom_tf>
   </plugin>
+  <plugin
+    filename="libgz-sim-joint-state-publisher-system.so"
+    name="gz::sim::systems::JointStatePublisher">
+    <topic>/joint_states</topic>
+  </plugin>
 </gazebo>
 <link name="base_link">
   <inertial>
-    <origin xyz="-0.12499450936127811 -0.0732393668268621 0.25843254250315395" rpy="0 0 0"/>
-    <mass value="11.269909330356606"/>
-    <inertia ixx="0.1243" iyy="0.218253" izz="0.256396" ixy="-2e-06" iyz="-0.0" ixz="3e-06"/>
+    <origin xyz="-0.12509032426168165 -0.07395516271652715 0.26127560952038015" rpy="0 0 0"/>
+    <mass value="21.041155080652292"/>
+    <inertia ixx="0.188108" iyy="0.289502" izz="0.293599" ixy="-0.000208" iyz="-0.000266" ixz="-7.4e-05"/>
   </inertial>
   <visual>
@@ -41,8 +46,14 @@
   </collision>
 </link>
-<link name="base_footprint"/>
+<joint name="base_footprint_joint" type="fixed">
+  <parent link="base_footprint"/>
+  <child link="base_link"/>
+  <origin xyz="0 0 0" rpy="0 0 0"/>
+</joint>
+<link name="base_footprint">
+</link>
 <link name="BHARAT_-FIH_-AMR-MAIN_WHEEL_WITH_MOTOR-PA-001__1__1">
   <inertial>
-    <origin xyz="7.392549115040059e-06 -0.04111510772339333 -1.6452849457837537e-07" rpy="0 0 0"/>
+    <origin xyz="7.392549115067815e-06 -0.04011510772339327 -1.6452849457837537e-07" rpy="0 0 0"/>
     <mass value="7.7692039603760845"/>
     <inertia ixx="0.01318" iyy="0.022658" izz="0.013179" ixy="-3e-06" iyz="0.0" ixz="0.0"/>
@@ -62,7 +73,47 @@
   </collision>
 </link>
+<link name="ball_caster_wheel__1__1">
+  <inertial>
+    <origin xyz="1.3877787807814457e-17 7.134979032596966e-08 -0.012099122560755626" rpy="0 0 0"/>
+    <mass value="0.1479113408447469"/>
+    <inertia ixx="2.2e-05" iyy="2e-05" izz="2.4e-05" ixy="0.0" iyz="0.0" ixz="-0.0"/>
+  </inertial>
+  <visual>
+    <origin xyz="-0.04 0.073241 -0.174741" rpy="0 0 0"/>
+    <geometry>
+      <mesh filename="file://$(find ros_project)/meshes/ball_caster_wheel__1__1.stl" scale="0.001 0.001 0.001"/>
+    </geometry>
+    <material name="silver"/>
+  </visual>
+  <collision>
+    <origin xyz="-0.04 0.073241 -0.174741" rpy="0 0 0"/>
+    <geometry>
+      <mesh filename="file://$(find ros_project)/meshes/ball_caster_wheel__1__1.stl" scale="0.001 0.001 0.001"/>
+    </geometry>
+  </collision>
+</link>
+<link name="ball_caster_wheel_1">
+  <inertial>
+    <origin xyz="-5.551115123125783e-17 7.134979036760303e-08 -0.012099122560755599" rpy="0 0 0"/>
+    <mass value="0.1479113408447469"/>
+    <inertia ixx="2.2e-05" iyy="2e-05" izz="2.4e-05" ixy="-0.0" iyz="0.0" ixz="-0.0"/>
+  </inertial>
+  <visual>
+    <origin xyz="0.29 0.073241 -0.174741" rpy="0 0 0"/>
+    <geometry>
+      <mesh filename="file://$(find ros_project)/meshes/ball_caster_wheel_1.stl" scale="0.001 0.001 0.001"/>
+    </geometry>
+    <material name="silver"/>
+  </visual>
+  <collision>
+    <origin xyz="0.29 0.073241 -0.174741" rpy="0 0 0"/>
+    <geometry>
+      <mesh filename="file://$(find ros_project)/meshes/ball_caster_wheel_1.stl" scale="0.001 0.001 0.001"/>
+    </geometry>
+  </collision>
+</link>
 <link name="BHARAT_-FIH_-AMR-MAIN_WHEEL_WITH_MOTOR-PA-001_1">
   <inertial>
-    <origin xyz="-7.3925491141657584e-06 0.04011525042358858 -1.6452849452286422e-07" rpy="0 0 0"/>
+    <origin xyz="-7.392549115026181e-06 0.040115250423588523 -1.6452849452286422e-07" rpy="0 0 0"/>
     <mass value="7.7692039603760845"/>
     <inertia ixx="0.01318" iyy="0.022658" izz="0.013179" ixy="-3e-06" iyz="-0.0" ixz="-0.0"/>
@@ -82,68 +133,24 @@
   </collision>
 </link>
-<link name="ball_caster_wheel__1__1">
-  <inertial>
-    <origin xyz="6.938893903907228e-18 7.135010103576089e-08 -0.012099122560755626" rpy="0 0 0"/>
-    <mass value="0.14791134084474702"/>
-    <inertia ixx="2.2e-05" iyy="2e-05" izz="2.4e-05" ixy="-0.0" iyz="-0.0" ixz="0.0"/>
-  </inertial>
-  <visual>
-    <origin xyz="-0.04 0.073241 -0.174741" rpy="0 0 0"/>
-    <geometry>
-      <mesh filename="file://$(find ros_project)/meshes/ball_caster_wheel__1__1.stl" scale="0.001 0.001 0.001"/>
-    </geometry>
-    <material name="silver"/>
-  </visual>
-  <collision>
-    <origin xyz="-0.04 0.073241 -0.174741" rpy="0 0 0"/>
-    <geometry>
-      <mesh filename="file://$(find ros_project)/meshes/ball_caster_wheel__1__1.stl" scale="0.001 0.001 0.001"/>
-    </geometry>
-  </collision>
-</link>
-<link name="ball_caster_wheel_1">
-  <inertial>
-    <origin xyz="0.0 7.135010100800532e-08 -0.012099122560755599" rpy="0 0 0"/>
-    <mass value="0.14791134084474702"/>
-    <inertia ixx="2.2e-05" iyy="2e-05" izz="2.4e-05" ixy="0.0" iyz="-0.0" ixz="0.0"/>
-  </inertial>
-  <visual>
-    <origin xyz="0.29 0.073241 -0.174741" rpy="0 0 0"/>
-    <geometry>
-      <mesh filename="file://$(find ros_project)/meshes/ball_caster_wheel_1.stl" scale="0.001 0.001 0.001"/>
-    </geometry>
-    <material name="silver"/>
-  </visual>
-  <collision>
-    <origin xyz="0.29 0.073241 -0.174741" rpy="0 0 0"/>
-    <geometry>
-      <mesh filename="file://$(find ros_project)/meshes/ball_caster_wheel_1.stl" scale="0.001 0.001 0.001"/>
-    </geometry>
-  </collision>
-</link>
-<link name="lidar_1">
-  <inertial>
-    <origin xyz="0.16 7.135009756631394e-08 0.01499992864990235" rpy="0 0 0"/>
-    <mass value="2.663442251713426"/>
-    <inertia ixx="0.002597" iyy="0.002597" izz="0.004794" ixy="0.0" iyz="0.0" ixz="0.0"/>
-  </inertial>
-  <visual>
-    <origin xyz="0.125 0.073241 -0.198241" rpy="0 0 0"/>
-    <geometry>
-      <mesh filename="file://$(find ros_project)/meshes/lidar_1.stl" scale="0.001 0.001 0.001"/>
-    </geometry>
-    <material name="silver"/>
-  </visual>
-  <collision>
-    <origin xyz="0.125 0.073241 -0.198241" rpy="0 0 0"/>
-    <geometry>
-      <mesh filename="file://$(find ros_project)/meshes/lidar_1.stl" scale="0.001 0.001 0.001"/>
-    </geometry>
-  </collision>
-</link>
-<joint name="base_joint" type="fixed">
-  <parent link="base_footprint"/>
-  <child link="base_link"/>
-</joint>
+<link name="Component1_1">
+  <inertial>
+    <origin xyz="0.195 7.13500976079473e-08 0.04331042864990181" rpy="0 0 0"/>
+    <mass value="0.5565046796809807"/>
+    <inertia ixx="0.000186" iyy="0.000186" izz="0.000341" ixy="-0.0" iyz="0.0" ixz="0.0"/>
+  </inertial>
+  <visual>
+    <origin xyz="0.125 0.073241 -0.296241" rpy="0 0 0"/>
+    <geometry>
+      <mesh filename="file://$(find ros_project)/meshes/Component1_1.stl" scale="0.001 0.001 0.001"/>
+    </geometry>
+    <material name="silver"/>
+  </visual>
+  <collision>
+    <origin xyz="0.125 0.073241 -0.296241" rpy="0 0 0"/>
+    <geometry>
+      <mesh filename="file://$(find ros_project)/meshes/Component1_1.stl" scale="0.001 0.001 0.001"/>
+    </geometry>
+  </collision>
+</link>
 <joint name="left_wheel_joint" type="continuous">
   <origin xyz="-0.125 -0.188241 0.226241" rpy="0 0 0"/>
@@ -152,4 +159,14 @@
   <axis xyz="0 1 0"/>
 </joint>
+<joint name="Rigid 3" type="fixed">
+  <origin xyz="0.04 -0.073241 0.174741" rpy="0 0 0"/>
+  <parent link="base_link"/>
+  <child link="ball_caster_wheel__1__1"/>
+</joint>
+<joint name="Rigid 4" type="fixed">
+  <origin xyz="-0.29 -0.073241 0.174741" rpy="0 0 0"/>
+  <parent link="base_link"/>
+  <child link="ball_caster_wheel_1"/>
+</joint>
 <joint name="right_wheel_joint" type="continuous">
   <origin xyz="-0.125 0.041759 0.226241" rpy="0 0 0"/>
@@ -158,24 +175,14 @@
   <axis xyz="0 1 0"/>
 </joint>
-<joint name="Rigid 3" type="fixed">
-  <origin xyz="0.04 -0.073241 0.174741" rpy="0 0 0"/>
-  <parent link="base_link"/>
-  <child link="ball_caster_wheel__1__1"/>
-</joint>
-<joint name="Rigid 4" type="fixed">
-  <origin xyz="-0.29 -0.073241 0.174741" rpy="0 0 0"/>
-  <parent link="base_link"/>
-  <child link="ball_caster_wheel_1"/>
-</joint>
-<joint name="Rigid 5" type="fixed">
-  <origin xyz="-0.125 -0.073241 0.198241" rpy="0 0 0"/>
-  <parent link="base_link"/>
-  <child link="lidar_1"/>
-</joint>
-<gazebo reference="lidar_1">
+<joint name="Rigid 7" type="fixed">
+  <origin xyz="-0.125 -0.073241 0.296241" rpy="0 0 0"/>
+  <parent link="base_link"/>
+  <child link="Component1_1"/>
+</joint>
+<gazebo reference="Component1_1">
   <sensor name="gpu_lidar" type="gpu_lidar">
     <pose>0 0 0 0 0 0</pose>
     <topic>/scan</topic>
-    <ignition_frame_id>lidar_1</ignition_frame_id>
+    <ignition_frame_id>Component1_1</ignition_frame_id>
     <update_rate>15</update_rate>
     <visualize>true</visualize>

File: src/ros_project/urdf1/materials.xacro (robot description, xacro)
@@ -1,4 +1,4 @@
 <?xml version="1.0" ?>
-<robot name="slam_lidar_midplate_front" xmlns:xacro="http://www.ros.org/wiki/xacro" >
+<robot name="slam" xmlns:xacro="http://www.ros.org/wiki/xacro" >
 <material name="silver">
   <color rgba="0.700 0.700 0.700 1.000"/>
